Commit message: professor th added

File: p_spombinho/p_spombinho_description/urdf/p_spombinho.gazebo.macro.xacro (robot description, xacro)
@@ -10,5 +10,5 @@
       <always_on>true</always_on>
       <contact>
-        <collision>base_footprint_fixed_joint_lump__base_link_collision_collision</collision>
+        <collision>base_footprint_fixed_joint_lump__base_link_collision</collision>
       </contact>
       <plugin name="base_link_contact_sensor_plugin" filename="libgazebo_ros_bumper.so">

Commit message: Back camera added as well as rviz changed

File: p_spombinho/p_spombinho_description/urdf/p_spombinho.gazebo.macro.xacro (robot description, xacro)
@@ -180,4 +180,37 @@
     </sensor>
   </gazebo>
+<!--    camera back -->
+  <gazebo reference="camera_rgb_frame_back">
+    <sensor type="camera" name="Pi Camera">
+      <always_on>true</always_on>
+      <visualize>${camera_visual}</visualize>
+      <camera>
+          <horizontal_fov>1.085595</horizontal_fov>
+          <image>
+              <width>1280</width>
+              <height>720</height>
+              <format>R8G8B8</format>
+          </image>
+          <clip>
+              <near>0.03</near>
+              <far>100</far>
+          </clip>
+      </camera>
+      <plugin name="camera_controller" filename="libgazebo_ros_camera.so">
+        <alwaysOn>true</alwaysOn>
+        <updateRate>30.0</updateRate>
+        <cameraName>camera_back</cameraName>
+        <frameName>camera_rgb_optical_frame</frameName>
+        <imageTopicName>rgb/image_raw</imageTopicName>
+        <cameraInfoTopicName>rgb/camera_info</cameraInfoTopicName>
+        <hackBaseline>0.07</hackBaseline>
+        <distortionK1>0.0</distortionK1>
+        <distortionK2>0.0</distortionK2>
+        <distortionK3>0.0</distortionK3>
+        <distortionT1>0.0</distortionT1>
+        <distortionT2>0.0</distortionT2>
+      </plugin>
+    </sensor>
+  </gazebo>
   </xacro:macro>
 </robot>

File: p_spombinho/p_spombinho_description/urdf/p_spombinho.urdf.xacro (robot description, xacro)
@@ -139,4 +139,5 @@
     </inertial>
   </link>
+<!--  imu -->
   <joint name="imu_joint" type="fixed">
     <parent link="base_link"/>
@@ -150,4 +151,5 @@
     <origin xyz="-0.064 0 0.122" rpy="0 0 0"/>
   </joint>
+<!--  laser scanner -->
   <link name="base_scan">
     <visual>
@@ -172,4 +174,5 @@
     </inertial>
   </link>
+<!--  camera front -->
   <joint name="camera_joint" type="fixed">
     <origin xyz="0.073 -0.011 0.084" rpy="0 0 0"/>
@@ -197,3 +200,29 @@
   </joint>
   <link name="camera_rgb_optical_frame"/>
+<!--  camera back   -->
+  <joint name="camera_joint_back" type="fixed">
+    <origin xyz="-0.2 -0.011 0.084" rpy="0 0 -3.14"/>
+    <parent link="base_link"/>
+    <child link="camera_link_back"/>
+  </joint>
+  <link name="camera_link_back">
+    <collision>
+      <origin xyz="0.005 0.011 0.013" rpy="0 0 0"/>
+      <geometry>
+        <box size="0.015 0.030 0.027"/>
+      </geometry>
+    </collision>
+  </link>
+  <joint name="camera_rgb_joint_back" type="fixed">
+    <origin xyz="0.003 0.011 0.009" rpy="0 0 0"/>
+    <parent link="camera_link_back"/>
+    <child link="camera_rgb_frame_back"/>
+  </joint>
+  <link name="camera_rgb_frame_back"/>
+  <joint name="camera_rgb_optical_joint_back" type="fixed">
+    <origin xyz="0 0 0" rpy="-1.57 0 -1.57"/>
+    <parent link="camera_rgb_frame_back"/>
+    <child link="camera_rgb_optical_frame_back"/>
+  </joint>
+  <link name="camera_rgb_optical_frame_back"/>
 </robot>
